File: NEC.kicad_pcb (KiCad board)
At the start: 2 copper layers, 314.3 x 76.2 mm, 123 parts, among them SW1 MX_SW_solder, SW10 MX_SW_solder, SW11 MX_SW_solder, SW12 MX_SW_solder, SW13 MX_SW_solder, SW14 MX_SW_solder, SW14(iso)1 MX_SW_solder, SW15 MX_SW_solder, SW16 MX_SW_solder, SW17 MX_SW_solder, SW18 MX_SW_solder, SW19 MX_SW_solder, SW2 MX_SW_solder, SW20 MX_SW_solder, SW21 MX_SW_solder, SW21(3)1 MX_SW_solder, SW22 MX_SW_solder, SW23 MX_SW_solder, SW24 MX_SW_solder, SW25 MX_SW_solder, SW26 MX_SW_solder, SW27 MX_SW_solder, SW28 MX_SW_solder, SW29 MX_SW_solder, SW3 MX_SW_solder, SW30 MX_SW_solder, SW31 MX_SW_solder, SW32 MX_SW_solder, SW33 MX_SW_solder, SW34 MX_SW_solder, SW35 MX_SW_solder, SW35(1.75)1 MX_SW_solder, SW36 MX_SW_solder, SW37 MX_SW_solder, SW37(1.75)1 MX_SW_solder, SW38 MX_SW_solder, SW39 MX_SW_solder, SW4 MX_SW_solder, SW40 MX_SW_solder, SW41 MX_SW_solder, SW42 MX_SW_solder, SW43 MX_SW_solder, SW44 MX_SW_solder, SW44(1.25)1 MX_SW_solder, SW45 MX_SW_solder, SW45(1.25)1 MX_SW_solder, SW46 MX_SW_solder, SW46(3)1 MX_SW_solder, SW47 MX_SW_solder, SW47(4)1 MX_SW_solder, SW48 MX_SW_solder, SW49 MX_SW_solder, SW49(3)1 MX_SW_solder, SW5 MX_SW_solder, SW50 MX_SW_solder, SW50(1.25)1 MX_SW_solder, SW51 MX_SW_solder, SW51(1.25)2 MX_SW_solder, SW52 RotaryEncoder_Switch, SW53 RotaryEncoder_Switch, SW6 MX_SW_solder, SW7 MX_SW_solder, SW8 MX_SW_solder, SW9 MX_SW_solder

Commit message: 1st draft compete
Parts:
- removed S7: MX_stab, marbastlib-mx:STAB_MX_P_6.25u
- removed SW47(4)1: MX_SW_solder, marbastlib-mx:SW_MX_1u
- added SW44(4)1: SW_Push_45deg, CherryMX:CherryMX_4.00u, F.Cu at (160.3, 88.9)
- added SW54: RotaryEncoder_Switch, marbastlib-various:ROT_Alps_EC11E-Switch, F.Cu at (136.5, 69.8)
- added SW55: RotaryEncoder_Switch, marbastlib-various:ROT_Alps_EC11E-Switch, F.Cu at (184.2, 69.8)
- moved D28 284.0 mm to (299.2, 55.7), turned to -90 degrees
- moved D43 284.0 mm to (306.4, 73.0), turned to -90 degrees
- moved D14 280.6 mm to (285.8, 36.4), turned to -90 degrees
- moved D13 269.2 mm to (273.1, 33.3), turned to -90 degrees
- moved D27 264.5 mm to (277.8, 52.4), turned to -90 degrees
- moved D42 261.5 mm to (282.6, 71.4), turned to -90 degrees
- moved D11 257.3 mm to (234.9, 33.3), turned to -90 degrees
- moved D12 249.3 mm to (254.0, 36.5), turned to -90 degrees
- moved D26 244.5 mm to (258.8, 55.6), turned to -90 degrees
- moved D41 241.4 mm to (263.5, 74.6), turned to -90 degrees
- moved D10 238.2 mm to (215.9, 36.5), turned to -90 degrees
- moved D25 227.5 mm to (239.7, 52.4), turned to -90 degrees
- moved D40 224.2 mm to (244.5, 71.4), turned to -90 degrees
- moved D9 223.4 mm to (196.8, 33.3), turned to -90 degrees
- moved D51 221.5 mm to (255.6, 90.5), turned to -90 degrees
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Connections:
- net Net-(D35-A) renamed row_2
- net Net-(D37-A) renamed row_4
- D7 pad 2: Net-(D7-A) -> row_1
- D8 pad 2: Net-(D8-A) -> row_3
- RZ1 pad 1: ROW0 -> ROW6
- RZ1 pad 10: LEFT_B -> COL1
- RZ1 pad 11: RIGHT_B -> COL2
- RZ1 pad 12: RIGHT_A -> COL3
- RZ1 pad 13: unconnected-(RZ1-GP12-Pad13) -> COL4
- RZ1 pad 14: COL6 -> LEFT_B
- RZ1 pad 15: COL5 -> LEFT_A
- RZ1 pad 16: COL4 -> RIGHT_A
- RZ1 pad 17: COL3 -> RIGHT_B
- RZ1 pad 18: COL2 -> COL5
- RZ1 pad 19: COL1 -> COL6
- RZ1 pad 2: ROW1 -> ROW7
- RZ1 pad 20: COL0 -> unconnected-(RZ1-GP29-Pad20)
- RZ1 pad 3: ROW2 -> ROW5
- RZ1 pad 4: ROW3 -> ROW4
- RZ1 pad 5: ROW4 -> ROW3
- RZ1 pad 6: ROW5 -> ROW2
- RZ1 pad 7: ROW6 -> COL0
- RZ1 pad 8: ROW7 -> ROW0
- RZ1 pad 9: LEFT_A -> ROW1
- SW44 pad 1: Net-(SW44(1.25)1-Pad1) -> COL1
- SW44(1.25)1 pad 1: Net-(SW44(1.25)1-Pad1) -> COL1
- SW52 pad S1: unconnected-(SW52-PadS1) -> row_1
- SW52 pad S2: unconnected-(SW52-PadS2) -> COL3
- SW53 pad S1: unconnected-(SW53-PadS1) -> row_3
- SW53 pad S2: unconnected-(SW53-PadS2) -> COL3
- SW7 pad 2: Net-(D7-A) -> row_1
- SW8 pad 2: Net-(D8-A) -> row_3
Routing:
- net COL4: track 0.00 -> 373.7 mm, vias 0 -> 1
- net ROW5: track 0.00 -> 370.1 mm
- net COL6: track 0.00 -> 366.9 mm, vias 0 -> 2
- net ROW6: track 0.00 -> 355.5 mm, vias 0 -> 1
- net COL5: track 0.00 -> 344.1 mm, vias 0 -> 2
- net ROW4: track 0.00 -> 337.9 mm
- net COL3: track 0.00 -> 332.3 mm, vias 0 -> 2
- net ROW3: track 0.00 -> 317.8 mm
- net ROW7: track 0.00 -> 313.4 mm, vias 0 -> 1
- net COL2: track 0.00 -> 309.0 mm, vias 0 -> 3
- net ROW2: track 0.00 -> 288.7 mm
- net ROW1: track 0.00 -> 269.7 mm
- net ROW0: track 0.00 -> 258.2 mm
- net COL1: track 0.00 -> 218.3 mm, vias 0 -> 2
- net RIGHT_B: track 0.00 -> 206.1 mm, vias 0 -> 3
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- added copper zone on B.Cu, net GND
- added copper zone on F.Cu, net GND
Other:
- board size 314.3 x 76.2 mm -> 314.3 x 77.5 mm
