File: NEC.kicad_sch (KiCad schematic)
At the start: 123 parts, among them SW1 MX_SW_solder, SW10 MX_SW_solder, SW11 MX_SW_solder, SW12 MX_SW_solder, SW13 MX_SW_solder, SW14 MX_SW_solder, SW14(iso)1 MX_SW_solder, SW15 MX_SW_solder, SW16 MX_SW_solder, SW17 MX_SW_solder, SW18 MX_SW_solder, SW19 MX_SW_solder, SW2 MX_SW_solder, SW20 MX_SW_solder, SW21 MX_SW_solder, SW21(3)1 MX_SW_solder, SW22 MX_SW_solder, SW23 MX_SW_solder, SW24 MX_SW_solder, SW25 MX_SW_solder, SW26 MX_SW_solder, SW27 MX_SW_solder, SW28 MX_SW_solder, SW29 MX_SW_solder, SW3 MX_SW_solder, SW30 MX_SW_solder, SW31 MX_SW_solder, SW32 MX_SW_solder, SW33 MX_SW_solder, SW34 MX_SW_solder, SW35 MX_SW_solder, SW35(1.75)1 MX_SW_solder, SW36 MX_SW_solder, SW37 MX_SW_solder, SW37(1.75)1 MX_SW_solder, SW38 MX_SW_solder, SW39 MX_SW_solder, SW4 MX_SW_solder, SW40 MX_SW_solder, SW41 MX_SW_solder, SW42 MX_SW_solder, SW43 MX_SW_solder, SW44 MX_SW_solder, SW44(1.25)1 MX_SW_solder, SW45 MX_SW_solder, SW45(1.25)1 MX_SW_solder, SW46 MX_SW_solder, SW46(3)1 MX_SW_solder, SW47 MX_SW_solder, SW47(4)1 MX_SW_solder, SW48 MX_SW_solder, SW49 MX_SW_solder, SW49(3)1 MX_SW_solder, SW5 MX_SW_solder, SW50 MX_SW_solder, SW50(1.25)1 MX_SW_solder, SW51 MX_SW_solder, SW51(1.25)2 MX_SW_solder, SW52 RotaryEncoder_Switch, SW53 RotaryEncoder_Switch, SW6 MX_SW_solder, SW7 MX_SW_solder, SW8 MX_SW_solder, SW9 MX_SW_solder

Commit message: 1st draft compete
Parts:
- removed S7: MX_stab, marbastlib-mx:STAB_MX_P_6.25u, symbol marbastlib-mx:MX_stab
- removed SW47(4)1: MX_SW_solder, marbastlib-mx:SW_MX_1u, symbol marbastlib-mx:MX_SW_solder
- added SW44(4)1: SW_Push_45deg, CherryMX:CherryMX_4.00u, symbol Switch:SW_Push_45deg
- added SW54, SW55: RotaryEncoder_Switch, marbastlib-various:ROT_Alps_EC11E-Switch, symbol Device:RotaryEncoder_Switch
Connections:
- net COL0: now also RZ1.7 (GP6); no longer RZ1.20 (GP29)
- net COL1: now also RZ1.10 (GP9), SW44(1.25)1.1, SW44.1; no longer RZ1.19 (GP28)
- net COL2: now also RZ1.11 (GP10), SW44(4)1.1; no longer RZ1.18 (GP27)
- net COL3: now also RZ1.12 (GP11), SW52.S2, SW53.S2, SW54.S2, SW55.S2; no longer RZ1.17 (GP26)
- net COL4: now also RZ1.13 (GP12); no longer RZ1.16 (GP15)
- net COL5: now also RZ1.18 (GP27); no longer RZ1.15 (GP14)
- net COL6: now also RZ1.19 (GP28); no longer RZ1.14 (GP13)
- net GND: now also SW54.C, SW55.C
- net LEFT_A: now also RZ1.15 (GP14), SW54.A; no longer RZ1.9 (GP8)
- net LEFT_B: now also RZ1.14 (GP13), SW54.B; no longer RZ1.10 (GP9)
- net RIGHT_A: now also RZ1.16 (GP15), SW55.A; no longer RZ1.12 (GP11)
- net RIGHT_B: now also RZ1.17 (GP26), SW55.B; no longer RZ1.11 (GP10)
- net ROW0: now also RZ1.8 (GP7); no longer RZ1.1 (GP0)
- net ROW1: now also RZ1.9 (GP8); no longer RZ1.2 (GP1)
- net ROW2: now also RZ1.6 (GP5); no longer RZ1.3 (GP2)
- net ROW3: now also RZ1.5 (GP4); no longer RZ1.4 (GP3)
- net ROW4: now also RZ1.4 (GP3); no longer RZ1.5 (GP4)
- net ROW5: now also RZ1.3 (GP2); no longer RZ1.6 (GP5)
- net ROW6: now also RZ1.1 (GP0); no longer RZ1.7 (GP6)
- net ROW7: now also RZ1.2 (GP1); no longer RZ1.8 (GP7)
- net row_4: now reaches D37.2 (A), SW37(1.75)1.2, SW37.2
- net row_4: now also SW55.S1
- net row_1: now reaches SW52.S1
- net row_1: now also D7.2 (A), SW7.2
- net row_3: now reaches SW53.S1
- net row_3: now also D8.2 (A), SW8.2
- net at D47.2 (A), SW47.2: now also SW44(4)1.2
- net row_2: now reaches D35.2 (A), SW35(1.75)1.2, SW35.2
- net row_2: now also SW54.S1
- no-connect marks 0 -> 1
Other:
- moved on the sheet: RZ1, S1, S2, S3, S4, S5, S6
