File: Project/NEC.kicad_sch (KiCad schematic)
At the start: 124 parts, among them SW1 MX_SW_solder, SW10 MX_SW_solder, SW11 MX_SW_solder, SW12 MX_SW_solder, SW13 MX_SW_solder, SW14 MX_SW_solder, SW14(iso)1 MX_SW_solder, SW15 MX_SW_solder, SW16 MX_SW_solder, SW17 MX_SW_solder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

Commit message: clearer labelling on THT diodes & fresh gerbers
Parts:
- D1, D10, D11, D12, D13, D14, D15, D16, D17, D18, D19, D2, D20, D21, D22, D23, D24, D25, D26, D27, D28, D29, D3, D30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: footprint Keebio-Parts:Diode-Hybrid-Back -> kbd:D3_TH_SMD_v2
